Commit message: fix wheel height in urdf

File: urdf/create2.urdf.xacro (robot description, xacro)
@@ -60,5 +60,5 @@
     <parent link="base_link"/>
     <child link="left_wheel_link"/>
-    <origin xyz="0 ${wheel_separation/2} 0" rpy="0 0 0"/>
+    <origin xyz="0 ${wheel_separation/2} -0.025" rpy="0 0 0"/>
     <axis xyz="0 1 0"/>
     <dynamics damping="0.2" friction="0.1"/>
@@ -88,5 +88,5 @@
     <parent link="base_link"/>
     <child link="right_wheel_link"/>
-    <origin xyz="0 ${-wheel_separation/2} 0" rpy="0 0 0"/>
+    <origin xyz="0 ${-wheel_separation/2} -0.025" rpy="0 0 0"/>
     <axis xyz="0 1 0"/>
     <dynamics damping="0.2" friction="0.1"/>

Commit message: add laser joint

File: urdf/create2.urdf.xacro (robot description, xacro)
@@ -142,3 +142,23 @@
     </ros2_control>
   </xacro:if>
+  <joint name="laser_joint" type="fixed">
+        <parent link="base_link"/>
+        <child link="laser_frame"/>
+        <origin xyz="0.122 0 0.08" rpy="0 0 0"/>
+    </joint>
+  <link name="laser_frame">
+      <visual>
+          <geometry>
+              <cylinder radius="0.03" length="0.025"/>
+          </geometry>
+          <material name="black"/>
+      </visual>
+      <visual>
+          <origin xyz="0 0 -0.025"/>
+          <geometry>
+            <box size="0.06 0.06 0.025"/>
+          </geometry>
+          <material name="black"/>
+      </visual>
+  </link>
 </robot>

Commit message: change laser frame name to match sllidar package

File: urdf/create2.urdf.xacro (robot description, xacro)
@@ -144,8 +144,8 @@
   <joint name="laser_joint" type="fixed">
         <parent link="base_link"/>
-        <child link="laser_frame"/>
+        <child link="laser"/>
         <origin xyz="0.122 0 0.08" rpy="0 0 0"/>
     </joint>
-  <link name="laser_frame">
+  <link name="laser">
       <visual>
           <geometry>

Commit message: rotate lidar frame 180 degrees

File: urdf/create2.urdf.xacro (robot description, xacro)
@@ -143,5 +143,5 @@
         <parent link="base_link"/>
         <child link="laser"/>
-        <origin xyz="0.122 0 0.08" rpy="0 0 0"/>
+        <origin xyz="0.122 0 0.08" rpy="0 0 3.1415"/>
     </joint>
   <link name="laser">
